File: OtterPill-CAN.sch (KiCad schematic (older format))
At the start: 18 parts, among them J1 pinh, J2 pinh, J3 CAN, J5 SWD, J7 PAD, U1 TJA1051T-3

Commit message: finalized schematic
Parts:
- removed D1: LED RED, LED_SMD:LED_0603_1608Metric, symbol Device:LED
- removed D2: LED GREEN, LED_SMD:LED_0603_1608Metric, symbol Device:LED
- removed R3, R4: 3k3, Resistor_SMD:R_0603_1608Metric, symbol Device:R
- J1: footprint Connector_PinHeader_2.54mm:PinHeader_1x04_P2.54mm_Vertical -> otter:PinHeader_1x04_P2.54mm_Vertical_NOSILK
- J2: footprint Connector_PinHeader_2.54mm:PinHeader_1x11_P2.54mm_Vertical -> otter:PinHeader_1x11_P2.54mm_Vertical_NOSILK
- J7: footprint Connector_PinHeader_2.54mm:PinHeader_1x01_P2.54mm_Vertical -> otter:PinHeader_1x01_P2.54mm_Vertical_NOSILK
Changed lines of the file:
@@
 F 0 "J7" H 4044 2675 50  0000 C CNN
 F 1 "PAD" H 4044 2766 50  0000 C CNN
-F 2 "Connector_PinHeader_2.54mm:PinHeader_1x01_P2.54mm_Vertical" H 4150 2900 50  0001 C CNN
+F 2 "otter:PinHeader_1x01_P2.54mm_Vertical_NOSILK" H 4150 2900 50  0001 C CNN
 F 3 "~" H 4150 2900 50  0001 C CNN
 	1    4150 2900
 	-1   0    0    1
-$EndComp
-$Comp
-L power:GND #PWR0114
-U 1 1 5CC79224
-P 5500 4750
-F 0 "#PWR0114" H 5500 4500 50  0001 C CNN
-F 1 "GND" H 5505 4577 50  0000 C CNN
-F 2 "" H 5500 4750 50  0001 C CNN
-F 3 "" H 5500 4750 50  0001 C CNN
-	1    5500 4750
-	1    0    0    -1
-$EndComp
-Wire Wire Line
-	5150 4750 5500 4750
-Wire Wire Line
-	5150 4450 5150 4350
-Wire Wire Line
-	5500 4450 5500 4350
-Connection ~ 5500 4750
-$Comp
-L Device:R R4
-U 1 1 5CC77C43
-P 5500 4600
-F 0 "R4" H 5570 4646 50  0000 L CNN
-F 1 "3k3" H 5570 4555 50  0000 L CNN
-F 2 "Resistor_SMD:R_0603_1608Metric" V 5430 4600 50  0001 C CNN
-F 3 "~" H 5500 4600 50  0001 C CNN
-	1    5500 4600
-	1    0    0    -1
-$EndComp
-$Comp
-L Device:R R3
-U 1 1 5CC777A1
-P 5150 4600
-F 0 "R3" H 5220 4646 50  0000 L CNN
-F 1 "3k3" H 5220 4555 50  0000 L CNN
-F 2 "Resistor_SMD:R_0603_1608Metric" V 5080 4600 50  0001 C CNN
-F 3 "~" H 5150 4600 50  0001 C CNN
-	1    5150 4600
-	1    0    0    -1
-$EndComp
-$Comp
-L Device:LED D2
-U 1 1 5CC77263
-P 5500 4200
-F 0 "D2" V 5539 4083 50  0000 R CNN
-F 1 "LED GREEN" V 5448 4083 50  0000 R CNN
-F 2 "LED_SMD:LED_0603_1608Metric" H 5500 4200 50  0001 C CNN
-F 3 "~" H 5500 4200 50  0001 C CNN
-	1    5500 4200
-	0    -1   -1   0
-$EndComp
-$Comp
-L Device:LED D1
-U 1 1 5CC766AA
-P 5150 4200
-F 0 "D1" V 5189 4083 50  0000 R CNN
-F 1 "LED RED" V 5098 4083 50  0000 R CNN
-F 2 "LED_SMD:LED_0603_1608Metric" H 5150 4200 50  0001 C CNN
-F 3 "~" H 5150 4200 50  0001 C CNN
-	1    5150 4200
-	0    -1   -1   0
 $EndComp
 $Comp
@@
 Text GLabel 9850 3450 0    50   Input ~ 0
 RXD
-Text GLabel 5500 4050 1    50   Input ~ 0
-TXD
-Text GLabel 5150 4050 1    50   Input ~ 0
-RXD
 Text GLabel 9850 2650 0    50   Input ~ 0
 413
@@
 F 0 "J1" H 8556 2828 50  0000 C CNN
 F 1 "pinh" H 8556 2737 50  0000 C CNN
-F 2 "Connector_PinHeader_2.54mm:PinHeader_1x04_P2.54mm_Vertical" H 8450 2550 50  0001 C CNN
+F 2 "otter:PinHeader_1x04_P2.54mm_Vertical_NOSILK" H 8450 2550 50  0001 C CNN
 F 3 "~" H 8450 2550 50  0001 C CNN
 	1    8450 2550
@@
 F 0 "J2" H 10023 2880 50  0000 R CNN
 F 1 "pinh" H 10023 2971 50  0000 R CNN
-F 2 "Connector_PinHeader_2.54mm:PinHeader_1x11_P2.54mm_Vertical" H 10050 2950 50  0001 C CNN
+F 2 "otter:PinHeader_1x11_P2.54mm_Vertical_NOSILK" H 10050 2950 50  0001 C CNN
 F 3 "~" H 10050 2950 50  0001 C CNN
 	1    10050 2950

Commit message: finalized layout
Parts:
- removed C1, C2: 100n 50V, Capacitor_SMD:C_0603_1608Metric, symbol Device:C_Small
- removed JP1: VIN, Jumper:SolderJumper-3_P1.3mm_Open_RoundedPad1.0x1.5mm, symbol Device:Jumper_NC_Dual
- removed JP2: WS2812, Jumper:SolderJumper-3_P1.3mm_Open_RoundedPad1.0x1.5mm, symbol Device:Jumper_NC_Dual
Connections:
- net CAN_H: now also R2.1, U1.7 (CANH)
- net CAN_L: now also R2.2, U1.6 (CANL)
Changed lines of the file:
@@
 	1    0    0    -1
 $EndComp
-Text GLabel 6900 2350 2    50   Input ~ 0
+Text GLabel 6650 2600 2    50   Input ~ 0
 CAN_H
-Text GLabel 6900 3050 2    50   Input ~ 0
+Text GLabel 6650 2800 2    50   Input ~ 0
 CAN_L
 $Comp
@@
 	-1   0    0    1
 $EndComp
-Text GLabel 6650 3300 3    50   Input ~ 0
-RXD
-$Comp
-L Device:Jumper_NC_Dual JP2
-U 1 1 5DB2C0C4
-P 6650 3050
-F 0 "JP2" V 6696 3152 50  0000 L CNN
-F 1 "WS2812" V 6605 3152 50  0000 L CNN
-F 2 "Jumper:SolderJumper-3_P1.3mm_Open_RoundedPad1.0x1.5mm" H 6650 3050 50  0001 C CNN
-F 3 "~" H 6650 3050 50  0001 C CNN
-	1    6650 3050
-	0    -1   -1   0
-$EndComp
 Connection ~ 6250 2800
 Wire Wire Line
-	6900 3050 6750 3050
-Wire Wire Line
 	6250 2800 6650 2800
-$Comp
-L Device:Jumper_NC_Dual JP1
-U 1 1 5DB2CF9D
-P 6650 2350
-F 0 "JP1" V 6696 2452 50  0000 L CNN
-F 1 "VIN" V 6605 2452 50  0000 L CNN
-F 2 "Jumper:SolderJumper-3_P1.3mm_Open_RoundedPad1.0x1.5mm" H 6650 2350 50  0001 C CNN
-F 3 "~" H 6650 2350 50  0001 C CNN
-	1    6650 2350
-	0    -1   -1   0
-$EndComp
 Wire Wire Line
 	6650 2600 6250 2600
 Connection ~ 6250 2600
-Text GLabel 6650 2100 1    50   Input ~ 0
-VIN
-Wire Wire Line
-	6900 2350 6750 2350
 $Comp
 L Device:R R5
@@
 	4500 2450 4400 2450
 $Comp
-L Device:C_Small C1
-U 1 1 5DB30195
-P 6350 1300
-F 0 "C1" H 6442 1346 50  0000 L CNN
-F 1 "100n 50V" H 6442 1255 50  0000 L CNN
-F 2 "Capacitor_SMD:C_0603_1608Metric" H 6350 1300 50  0001 C CNN
-F 3 "~" H 6350 1300 50  0001 C CNN
-	1    6350 1300
-	1    0    0    -1
-$EndComp
-$Comp
-L power:GND #PWR0103
-U 1 1 5DB301A2
-P 6350 1400
-F 0 "#PWR0103" H 6350 1150 50  0001 C CNN
-F 1 "GND" H 6355 1227 50  0000 C CNN
-F 2 "" H 6350 1400 50  0001 C CNN
-F 3 "" H 6350 1400 50  0001 C CNN
-	1    6350 1400
-	1    0    0    -1
-$EndComp
-Text GLabel 6350 1200 1    50   Input ~ 0
-VIN
-$Comp
-L Device:C_Small C2
-U 1 1 5DB30CB8
-P 6900 1300
-F 0 "C2" H 6992 1346 50  0000 L CNN
-F 1 "100n 50V" H 6992 1255 50  0000 L CNN
-F 2 "Capacitor_SMD:C_0603_1608Metric" H 6900 1300 50  0001 C CNN
-F 3 "~" H 6900 1300 50  0001 C CNN
-	1    6900 1300
-	1    0    0    -1
-$EndComp
-$Comp
-L power:GND #PWR0105
-U 1 1 5DB30CBF
-P 6900 1400
-F 0 "#PWR0105" H 6900 1150 50  0001 C CNN
-F 1 "GND" H 6905 1227 50  0000 C CNN
-F 2 "" H 6900 1400 50  0001 C CNN
-F 3 "" H 6900 1400 50  0001 C CNN
-	1    6900 1400
-	1    0    0    -1
-$EndComp
-Text GLabel 6900 1200 1    50   Input ~ 0
-VIN
-$Comp
 L Connector_Generic_MountingPin:Conn_01x03_MountingPin J3
